Commit message: Rover with real dimensions

File: ardupilot_sitl_gazebo_plugin/urdf/rover.urdf (robot description, URDF)
Before this commit: robot rover, 7 links, 6 joints
Links:
- link chassis: geometry collision box size=0.268 0.2 0.012; visual mesh filename=package://ardupilot_sitl_gazebo_plugin/meshes/meshes_rover/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 scale=0.0011 0.0011 0.0011
- link front_left_wheel: geometry collision cylinder length=0.05588 radius=0.0635; visual mesh filename=package://ardupilot_sitl_gazebo_plugin/meshes/meshes_rover/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 scale=0.0014 0.0014 0.0014
- link front_right_wheel: geometry collision cylinder length=0.05588 radius=0.0635; visual mesh filename=package://ardupilot_sitl_gazebo_plugin/meshes/meshes_rover/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 scale=0.0014 0.0014 0.0014
- link rear_left_wheel: geometry collision cylinder length=0.05588 radius=0.0635; visual mesh filename=package://ardupilot_sitl_gazebo_plugin/meshes/meshes_rover/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 scale=0.0014 0.0014 0.0014
- link rear_right_wheel: geometry collision cylinder length=0.05588 radius=0.0635; visual mesh filename=package://ardupilot_sitl_gazebo_plugin/meshes/meshes_rover/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 scale=0.0014 0.0014 0.0014
Joints:
- joint front_left_steering_joint: origin xyz=1.20222  0.5 0.35515 rpy=-1.52 0 0 -> xyz=0.240444 0.1 0.07103 rpy=-1.52 0 0
- joint front_left_wheel_joint: origin xyz=0 0 0.21562 rpy=0 0 0 -> xyz=0.0 0.0 0.043124 rpy=0 0 0
- joint front_right_steering_joint: origin xyz=1.20222 -0.5 0.35515 rpy=1.52 0 0 -> xyz=0.240444 -0.1 0.07103 rpy=1.52 0 0
- joint front_right_wheel_joint: origin xyz=0 0 0.21562 rpy=0 0 0 -> xyz=0.0 0.0 0.043124 rpy=0 0 0
- joint rear_left_wheel_joint: origin xyz=-0.75 0.75 0.34697 rpy=-1.52 0 0 -> xyz=-0.15 0.15 0.069394 rpy=-1.52 0 0
- joint rear_right_wheel_joint: origin xyz=-0.75 -0.75 0.34697 rpy=1.52 0 0 -> xyz=-0.15 -0.15 0.069394 rpy=1.52 0 0
